File: KiCad/SEM/SEM.kicad_pcb (KiCad board)
At the start: 2 copper layers, 64.5 x 56.2 mm, 23 parts, among them J1 RJ12, J2 FPC_01x10, J3 Micro_SD_Card, J4 Conn_01x03_Female, J5 Raspberry_Pi_2_3, Q1 DMP3056LSD, SW1 RotaryEncoder_Switch, U1 L78L33_TO252, U2 ESP32-WROOM-32

Commit message: KiCAD update
Parts:
- removed J5: Raspberry_Pi_2_3, Connector_PinHeader_1.27mm:PinHeader_2x20_P1.27mm_Vertical
- removed Q1: DMP3056LSD, Package_SO:Diodes_SO-8EP
- removed SW1: RotaryEncoder_Switch, Connector_PinHeader_2.00mm:PinHeader_2x03_P2.00mm_Vertical
- added C7: 10u, Capacitor_SMD:C_1206_3216Metric, F.Cu at (148.1, 63.4)
- added R7: 10K, Resistor_SMD:R_0603_1608Metric, F.Cu at (154.6, 79.1)
- added U3: AMS1117-3.3, Package_TO_SOT_SMD:SOT-223-3_TabPin2, F.Cu at (128.9, 61.5)
- added U4: ESP32-WROOM-32, RF_Module:ESP32-WROOM-32, F.Cu at (165.9, 70.0)
- C2: value 0.33u -> 10u; footprint Capacitor_SMD:C_0805_2012Metric_Pad1.18x1.45mm_HandSolder -> Capacitor_SMD:C_1206_3216Metric
- C3: value 100u -> 1u; footprint Capacitor_SMD:C_1206_3216Metric -> Capacitor_SMD:C_1812_4532Metric
- C6: value 100u -> 22u; footprint Capacitor_SMD:C_1206_3216Metric -> Capacitor_SMD:C_1812_4532Metric
- J1: value RJ12 -> FPC_01x10; footprint Connector_RJ:RJ12_Amphenol_54601 -> Connector_FFC-FPC:Hirose_FH12-10S-0.5SH_1x10-1MP_P0.50mm_Horizontal
- J2: value FPC_01x10 -> RJ12; footprint Connector_FFC-FPC:Hirose_FH12-10S-0.5SH_1x10-1MP_P0.50mm_Horizontal -> Connector_RJ:RJ12_Amphenol_54601
- J4: value Conn_01x03_Female -> USB_B_Micro; footprint Connector_PinHeader_1.27mm:PinHeader_1x03_P1.27mm_Horizontal -> Connector_USB:USB_Micro-B_Molex-105017-0001
- R3: value 10K -> 330R
- U1: value L78L33_TO252 -> ACPL-214-500E; footprint Package_TO_SOT_SMD:TO-252-2 -> Package_SO:SOP-4_4.4x2.6mm_P1.27mm
- U2: value ESP32-WROOM-32 -> 6N137; footprint RF_Module:ESP32-WROOM-32 -> Package_DIP:DIP-8_W7.62mm
- moved C6 54.9 mm to (126.1, 68.6), turned to 180 degrees
- moved J4 45.7 mm to (145.8, 50.9)
- moved J2 35.5 mm to (138.8, 88.7), turned to -90 degrees
- moved C2 29.8 mm to (133.2, 73.0)
- moved R4 29.3 mm to (152.5, 90.7)
- moved R3 29.2 mm to (138.0, 101.2)
- moved C4 28.6 mm to (133.3, 68.6), turned to 0 degrees
- moved U2 28.5 mm to (142.6, 94.8)
- moved C5 21.7 mm to (151.5, 63.4), turned to -90 degrees
- moved C1 18.7 mm to (160.0, 93.7)
- moved J3 13.2 mm to (171.5, 96.8)
- moved D1 9.74 mm to (180.8, 84.4)
- moved R1 9.62 mm to (180.8, 81.5)
- moved U1 9.56 mm to (146.6, 90.0), turned to 180 degrees
- moved D2 9.28 mm to (184.2, 84.4)
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Connections:
- C1 pad 1: +5V -> +3V3
- C3 pad 1: +3V3 -> RST
- C4 pad 1: +3V3 -> +5V
- J1 pad 1: +5V -> GND
- J1 pad 2: Net-(J1-Pad2) -> GND
- J1 pad 3: unconnected-(J1-Pad3) -> RST
- J1 pad 4: unconnected-(J1-Pad4) -> BOOT
- J1 pad 5: Net-(J1-Pad5) -> RXP
- J1 pad 6: GND -> RX0
- J2 pad 1: GND -> +5VA
- J2 pad 2: GND -> Net-(J2-Pad2)
- J2 pad 3: RST -> unconnected-(J2-Pad3)
- J2 pad 4: BOOT -> unconnected-(J2-Pad4)
- J2 pad 5: RX0 -> Net-(J2-Pad5)
- J2 pad 6: TX0 -> GND1
- J4 pad 1: GND -> +5V
- J4 pad 2: +5V -> unconnected-(J4-Pad2)
- J4 pad 3: GND -> unconnected-(J4-Pad3)
- R3 pad 1: +3V3 -> +5VA
- R3 pad 2: Data -> Net-(R3-Pad2)
- R4 pad 1: +5V -> Net-(R4-Pad1)
- R4 pad 2: Net-(J1-Pad2) -> Request
- U1 pad 1: +3V3 -> Net-(R4-Pad1)
- U1 pad 3: +5V -> Net-(J2-Pad2)
- U2 pad 1: GND -> unconnected-(U2-Pad1)
- U2 pad 2: +3V3 -> Net-(R3-Pad2)
- U2 pad 3: RST -> Net-(J2-Pad5)
- U2 pad 4: unconnected-(U2-Pad4) -> (no net)
- U2 pad 5: unconnected-(U2-Pad5) -> GND
- U2 pad 6: unconnected-(U2-Pad6) -> Data
- U2 pad 7: unconnected-(U2-Pad7) -> GND
- U2 pad 8: unconnected-(U2-Pad8) -> +3V3
Routing:
- net +3V3: track 157.5 -> 14.1 mm, vias 6 -> 0
- net +5V: track 109.3 -> 0.00 mm
- net GND: track 106.2 -> 36.4 mm, vias 24 -> 12
- net VSPI-SCLK: track 78.7 -> 26.1 mm, vias 4 -> 2
- net Rotary_Sw: track 50.9 -> 0.00 mm, vias 1 -> 0
- net RST: track 49.5 -> 4.20 mm, vias 2 -> 0
- net Rotary_B: track 43.5 -> 0.00 mm, vias 1 -> 0
- net Rotary_A: track 42.1 -> 0.00 mm, vias 1 -> 0
- net VSPI-MOSI: track 74.7 -> 34.1 mm
- net TX0: track 32.2 -> 0.00 mm, vias 2 -> 0
- net RX0: track 30.4 -> 0.00 mm, vias 2 -> 0
- net Request: track 27.8 -> 0.00 mm
- net GPIO16: track 24.5 -> 0.00 mm
- net Data: track 23.7 -> 0.00 mm
- net E-DC: track 23.5 -> 0.00 mm
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Other:
- outline, holes or cut-outs redrawn
