File: KiCad/SEM/SEM.kicad_sch (KiCad schematic)
At the start: 32 parts, among them J1 RJ12, J2 FPC_01x10, J3 Micro_SD_Card, J4 Conn_01x03_Female, J5 Raspberry_Pi_2_3, SW1 RotaryEncoder_Switch, U1 AMS1117-3.3, U2 ESP32-WROOM-32

Commit message: KiCAD update
Parts:
- removed C6: 10u, Capacitor_SMD:C_1206_3216Metric, symbol Device:C_Small
- removed C? (x3): 0.1u, Capacitor_SMD:C_1812_4532Metric, symbol Device:C_Small
- removed C?: 1u, Capacitor_SMD:C_1812_4532Metric, symbol Device:C_Small
- removed J4: Conn_01x03_Female, Connector_PinHeader_2.54mm:PinHeader_1x03_P2.54mm_Vertical, symbol Connector:Conn_01x03_Female
- removed J5: Raspberry_Pi_2_3, Connector_PinHeader_2.54mm:PinHeader_2x40_P2.54mm_Vertical, symbol Connector:Raspberry_Pi_2_3
- removed JP? (x2): SolderJumper_3_Bridged12, symbol Jumper:SolderJumper_3_Bridged12
- removed Q?: BUK7M6R3-40EX, Package_TO_SOT_SMD:LFPAK33, symbol Transistor_FET:BUK7M6R3-40EX
- removed R? (x3): 10K, Resistor_SMD:R_0603_1608Metric, symbol Device:R_Small
- removed SW1: RotaryEncoder_Switch, Connector_PinHeader_2.00mm:PinHeader_2x03_P2.00mm_Vertical, symbol Device:RotaryEncoder_Switch
- removed U2: ESP32-WROOM-32, RF_Module:ESP32-WROOM-32, symbol RF_Module:ESP32-WROOM-32
- removed U?: (no value), symbol 74xGxx:74AHC1G126
- added C5: 0.1u, Capacitor_SMD:C_1812_4532Metric, symbol Device:C_Small
- added C7: 10u, Capacitor_SMD:C_1206_3216Metric, symbol Device:C_Small
- added J4: USB_B_Micro, Connector_USB:USB_Micro-B_Molex-105017-0001, symbol Connector:USB_B_Micro
- added R6, R7: 10K, Resistor_SMD:R_0603_1608Metric, symbol Device:R_Small
- added U1: ACPL-214-500E, Package_SO:SOP-4_4.4x2.6mm_P1.27mm, symbol Isolator:ACPL-214-500E
- added U2: 6N137, Package_DIP:DIP-8_W7.62mm, symbol Isolator:6N137
- added U4: ESP32-WROOM-32, RF_Module:ESP32-WROOM-32, symbol RF_Module:ESP32-WROOM-32
- C3: value 10u -> 1u; footprint Capacitor_SMD:C_1206_3216Metric -> Capacitor_SMD:C_1812_4532Metric
- R3: value 10K -> 330R
- gave numbers to parts that had none: 2
- renumbered C5 to C1, C4 to C6, J2 to J1, J1 to J2, U1 to U3
Connections:
- net TXP is gone; now on net RX0: J1.6 (Pin_6)
- net +3V3: now also C5.1, C7.1, R6.1, U2.8 (VCC), U4.2 (VDD); no longer C3.1, R3.1
- net +5V: now also J4.1 (VBUS); no longer C1.2, C2.2, C3.2, C4.2, C6.2, D1.1 (K), D2.1 (K), J1.1 (Pin_1), J1.2 (Pin_2), J1.7 (Pin_7), J2.1, J2.6, J3.6 (VSS), J3.9 (SHIELD), R4.1, U3.1 (GND)
- net BOOT: now also R6.2, U4.25 (IO0)
- net Data: now also U2.6 (VO), U4.13 (IO14); no longer J2.5, R3.2
- net E-Busy: now also U4.29 (IO5)
- net E-CS: now also U4.8 (IO32)
- net E-DC: now also U4.33 (IO21)
- net E-RST: now also U4.36 (IO22)
- net GPIO16: now also U4.27 (IO16)
- net LED_ACT: now also U4.24 (IO2)
- net RST: now also C3.1, U4.3 (EN)
- net RX0: now also U4.34 (RXD0/IO3)
- net RXP: now also U4.35 (TXD0/IO1)
- net Request: now also R4.2, U4.16 (IO13)
- net Rotary_A: now also U4.11 (IO26)
- net Rotary_B: now also U4.12 (IO27)
- net Rotary_Sw: now also U4.10 (IO25)
- net SD-CS: now also U4.28 (IO17)
- net VSPI-MISO: now also U4.31 (IO19)
- net VSPI-MOSI: now also U4.37 (IO23)
- net VSPI-SCLK: now also U4.30 (IO18)
- net at J2.2: now also U1.3
- new net: J2.5, U2.3 (C)
- new net: R4.1, U1.1
- new net: R7.1, U4.14 (IO12)
- new net: R3.2, U2.2 (A)
- new net +5VA: J2.1, R3.1, U1.4
- new net GND: C1.2, C2.2, C3.2, C4.2, C5.2, C6.2, C7.2, D1.1 (K), D2.1 (K), J1.1 (Pin_1), J1.2 (Pin_2), J1.7 (Pin_7), J3.6 (VSS), J3.9 (SHIELD), J4.5 (GND), R7.2, U1.2, U2.5 (GND), U2.7 (EN), U3.1 (GND), U4.1 (GND), U4.15 (GND), U4.38 (GND), U4.39 (GND)
- new net GND1: J2.6
- no-connect marks 41 -> 22
Other:
- note added: "USB 5V power in"
- note removed: "Connectino to Epaper Display"
- note removed: "Possible 5V input"
- note removed: "Rotary Encoder"
- moved on the sheet: C1, C2, C4, C6, D1, D2, J1, J3, R1, R2, U3
