File: KiCad/SEM2/SEM2.kicad_pcb (KiCad board)
At the start: 2 copper layers, 52.8 x 52.3 mm, 6 parts, among them J1 RJ12, J2 Micro_SD_Card, U1 6N137, U2 ESP32-DevBoard

Commit message: Update KiCAD design
Connections:
- J1 pad 1: GND1 -> +5VA
- J1 pad 2: Net-(U1-Pad3) -> +5VA
- J1 pad 3: unconnected-(J1-Pad3) -> GND1
- J1 pad 4: GND1 -> unconnected-(J1-Pad4)
- J1 pad 5: +5VA -> Net-(U1-Pad3)
- J1 pad 6: +5VA -> GND1
Routing:
- net Net-(U1-Pad3): track 14.3 -> 28.2 mm
- net +5VA: track 25.7 -> 22.1 mm
Changed lines of the file:
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@@
   (net 3 "+5VA")
   (net 4 "GND1")
-  (net 5 "unconnected-(J1-Pad3)")
+  (net 5 "unconnected-(J1-Pad4)")
   (net 6 "Net-(U1-Pad3)")
   (net 7 "unconnected-(J2-Pad1)")
@@
     (pad "" np_thru_hole circle (at 8.25 8.89 90) (size 3.25 3.25) (drill 3.25) (layers *.Cu *.Mask))
     (pad "1" thru_hole rect (at 0 0 90) (size 1.52 1.52) (drill 0.76) (layers *.Cu *.Mask)
+      (net 3 "+5VA") (pintype "passive"))
+    (pad "2" thru_hole circle (at 1.27 2.54 90) (size 1.52 1.52) (drill 0.76) (layers *.Cu *.Mask)
+      (net 3 "+5VA") (pintype "passive"))
+    (pad "3" thru_hole circle (at 2.54 0 90) (size 1.52 1.52) (drill 0.76) (layers *.Cu *.Mask)
       (net 4 "GND1") (pintype "passive"))
-    (pad "2" thru_hole circle (at 1.27 2.54 90) (size 1.52 1.52) (drill 0.76) (layers *.Cu *.Mask)
+    (pad "4" thru_hole circle (at 3.81 2.54 90) (size 1.52 1.52) (drill 0.76) (layers *.Cu *.Mask)
+      (net 5 "unconnected-(J1-Pad4)") (pintype "passive+no_connect"))
+    (pad "5" thru_hole circle (at 5.08 0 90) (size 1.52 1.52) (drill 0.76) (layers *.Cu *.Mask)
       (net 6 "Net-(U1-Pad3)") (pintype "passive"))
-    (pad "3" thru_hole circle (at 2.54 0 90) (size 1.52 1.52) (drill 0.76) (layers *.Cu *.Mask)
-      (net 5 "unconnected-(J1-Pad3)") (pintype "passive+no_connect"))
-    (pad "4" thru_hole circle (at 3.81 2.54 90) (size 1.52 1.52) (drill 0.76) (layers *.Cu *.Mask)
+    (pad "6" thru_hole circle (at 6.35 2.54 90) (size 1.52 1.52) (drill 0.76) (layers *.Cu *.Mask)
       (net 4 "GND1") (pintype "passive"))
-    (pad "5" thru_hole circle (at 5.08 0 90) (size 1.52 1.52) (drill 0.76) (layers *.Cu *.Mask)
-      (net 3 "+5VA") (pintype "passive"))
-    (pad "6" thru_hole circle (at 6.35 2.54 90) (size 1.52 1.52) (drill 0.76) (layers *.Cu *.Mask)
-      (net 3 "+5VA") (pintype "passive"))
     (model "${KICAD6_3DMODEL_DIR}/Connector_RJ.3dshapes/RJ12_Amphenol_54601.wrl"
       (offset (xyz 0 0 0))
@@
   (segment (start 135.2804 80.9752) (end 142.367 80.9752) (width 0.25) (layer "B.Cu") (net 2))
   (segment (start 138.9888 83.1836) (end 136.7804 80.9752) (width 0.25) (layer "B.Cu") (net 2))
-  (segment (start 155.7396 87.376) (end 155.7396 68.9404) (width 0.25) (layer "F.Cu") (net 3))
-  (segment (start 155.7396 68.9404) (end 152.758 65.9588) (width 0.25) (layer "F.Cu") (net 3))
-  (segment (start 152.758 65.9588) (end 152.7022 66.0146) (width 0.25) (layer "B.Cu") (net 3))
-  (segment (start 152.7022 66.0146) (end 151.4322 66.0146) (width 0.25) (layer "B.Cu") (net 3))
-  (segment (start 151.4322 66.0146) (end 150.218 67.2288) (width 0.25) (layer "B.Cu") (net 3))
-  (segment (start 151.673 70.8538) (end 150.218 72.3088) (width 0.25) (layer "B.Cu") (net 4))
-  (segment (start 151.673 69.5838) (end 151.673 70.8538) (width 0.25) (layer "B.Cu") (net 4))
-  (segment (start 152.758 68.4988) (end 151.673 69.5838) (width 0.25) (layer "B.Cu") (net 4))
-  (segment (start 150.0532 83.5814) (end 151.221 83.5814) (width 0.25) (layer "B.Cu") (net 6))
-  (segment (start 151.221 83.5814) (end 152.758 82.0444) (width 0.25) (layer "B.Cu") (net 6))
-  (segment (start 152.758 71.0388) (end 152.758 82.0444) (width 0.25) (layer "B.Cu") (net 6))
+  (segment (start 155.6258 71.374) (end 155.2906 71.0388) (width 0.25) (layer "F.Cu") (net 3))
+  (segment (start 155.2906 71.0388) (end 152.758 71.0388) (width 0.25) (layer "F.Cu") (net 3))
+  (segment (start 155.7396 87.376) (end 155.6258 87.2622) (width 0.25) (layer "F.Cu") (net 3))
+  (segment (start 155.6258 87.2622) (end 155.6258 71.374) (width 0.25) (layer "F.Cu") (net 3))
+  (segment (start 151.488 71.0388) (end 150.218 72.3088) (width 0.25) (layer "B.Cu") (net 3))
+  (segment (start 152.758 71.0388) (end 151.488 71.0388) (width 0.25) (layer "B.Cu") (net 3))
+  (segment (start 151.673 68.3138) (end 150.218 69.7688) (width 0.25) (layer "B.Cu") (net 4))
+  (segment (start 151.673 67.0438) (end 151.673 68.3138) (width 0.25) (layer "B.Cu") (net 4))
+  (segment (start 152.758 65.9588) (end 151.673 67.0438) (width 0.25) (layer "B.Cu") (net 4))
+  (segment (start 150.218 65.7074) (end 151.5618 64.3636) (width 0.25) (layer "B.Cu") (net 6))
+  (segment (start 154.8638 65.1002) (end 154.8638 79.9386) (width 0.25) (layer "B.Cu") (net 6))
+  (segment (start 150.218 67.2288) (end 150.218 65.7074) (width 0.25) (layer "B.Cu") (net 6))
+  (segment (start 154.8638 79.9386) (end 151.221 83.5814) (width 0.25) (layer "B.Cu") (net 6))
+  (segment (start 154.1272 64.3636) (end 154.8638 65.1002) (width 0.25) (layer "B.Cu") (net 6))
+  (segment (start 151.221 83.5814) (end 150.0532 83.5814) (width 0.25) (layer "B.Cu") (net 6))
+  (segment (start 151.5618 64.3636) (end 154.1272 64.3636) (width 0.25) (layer "B.Cu") (net 6))
   (segment (start 137.4394 105.4354) (end 138.9204 106.9164) (width 0.25) (layer "F.Cu") (net 8))
   (segment (start 137.4394 91.8972) (end 137.4394 105.4354) (width 0.25) (layer "F.Cu") (net 8))
