File: KiCad/SEM2/SEM2.kicad_sch (KiCad schematic)
At the start: 6 parts, among them J1 RJ12, J2 Micro_SD_Card, U1 6N137, U2 ESP32-DevBoard

Commit message: Update KiCAD design
Connections:
- net +5VA: now also J1.1, J1.2; no longer J1.5, J1.6
- net GND1: now also J1.3, J1.6; no longer J1.1, J1.4
- net at U1.3 (C): now also J1.5; no longer J1.2
Other:
- company: (none) -> Sani7
- title: (none) -> Data reading circuit
Changed lines of the file:
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@@
 (kicad_sch (version 20211123) (generator eeschema)
   (paper "A4")
+  (title_block
+    (title "Data reading circuit")
+    (rev "2")
+    (company "Sani7")
+    (comment 1 "github.com/Sani7/SEM")
+    (comment 2 "(c) Sander Speetjens")
+  )
   (junction (at 43.18 27.94) (diameter 0) (color 0 0 0 0)
   )
@@
     )
     (pin "1")
-  )
-  (symbol (lib_id "Connector:RJ12") (at 30.48 35.56 0) (unit 1)
-    (in_bom yes) (on_board yes)
-    (property "Reference" "J1" (id 0) (at 22.1234 35.4584 0)
-      (effects (font (size 1.27 1.27)) (justify right))
-    )
-    (property "Value" "RJ12" (id 1) (at 22.1234 33.147 0)
-      (effects (font (size 1.27 1.27)) (justify right))
-    )
-    (property "Footprint" "Connector_RJ:RJ12_Amphenol_54601" (id 2) (at 30.48 34.925 90)
-      (effects (font (size 1.27 1.27)) hide)
-    )
-    (property "Datasheet" "2135977" (id 3) (at 30.48 34.925 90)
-      (effects (font (size 1.27 1.27)) hide)
-    )
-    (pin "1")
-    (pin "2")
-    (pin "3")
-    (pin "4")
-    (pin "5")
-    (pin "6")
   )
   (symbol (lib_id "power:GND") (at 21.59 77.47 0) (unit 1)
@@
     (pin "9")
   )
+  (symbol (lib_id "Connector:RJ12") (at 30.48 33.02 0) (mirror x) (unit 1)
+    (in_bom yes) (on_board yes)
+    (property "Reference" "J1" (id 0) (at 22.1234 33.1216 0)
+      (effects (font (size 1.27 1.27)) (justify right))
+    )
+    (property "Value" "RJ12" (id 1) (at 22.1234 35.433 0)
+      (effects (font (size 1.27 1.27)) (justify right))
+    )
+    (property "Footprint" "Connector_RJ:RJ12_Amphenol_54601" (id 2) (at 30.48 33.655 90)
+      (effects (font (size 1.27 1.27)) hide)
+    )
+    (property "Datasheet" "2135977" (id 3) (at 30.48 33.655 90)
+      (effects (font (size 1.27 1.27)) hide)
+    )
+    (pin "1")
+    (pin "2")
+    (pin "3")
+    (pin "4")
+    (pin "5")
+    (pin "6")
+  )
   (symbol (lib_id "power:+5VA") (at 43.18 26.035 0) (unit 1)
     (in_bom yes) (on_board yes)
@@
       (reference "C1") (unit 1) (value "0.1u") (footprint "Capacitor_SMD:C_1812_4532Metric")
     )
-    (path "/67ca49af-04af-4784-aec0-2ab4a28ac61d"
+    (path "/d83f6d9f-8b2f-4436-8bd7-ccdd6381d75c"
       (reference "J1") (unit 1) (value "RJ12") (footprint "Connector_RJ:RJ12_Amphenol_54601")
     )
